File: schematics/kicad/LVL_SHIFT_3_TO_5.sch (KiCad schematic (older format))
At the start: 3 parts

Commit message: Change a lot of things, especially pinning between sheets
Parts:
- added U11, U12: 74AHC125, symbol 74AHC125
- gave numbers to parts that had none: 3
Connections:
- net +5V: now also U11.14 (VCC), U12.14 (VCC)
- net GND: now also U11.1 (/1OE), U11.10 (/3OE), U11.13 (/4OE), U11.4 (/2OE), U11.7 (GND), U12.1 (/1OE), U12.10 (/3OE), U12.13 (/4OE), U12.4 (/2OE), U12.7 (GND)
- net RAM_WE_5V: now reaches U10.11 (4Y)
- net RAM_WE_3V: now reaches U10.12 (4A)
- net RAM_OE_5V: now reaches U10.8 (3Y)
- net RAM_OE_3V: now reaches U10.9 (3A)
- new net CS_PERIPH_0_3V: U11.2 (1A)
- new net CS_PERIPH_0_5V: U11.3 (1Y)
- new net CS_PERIPH_1_3V: U11.5 (2A)
- new net CS_PERIPH_1_5V: U11.6 (2Y)
- new net CS_PERIPH_2_3V: U11.9 (3A)
- new net CS_PERIPH_2_5V: U11.8 (3Y)
- new net CS_PERIPH_3_3V: U11.12 (4A)
- new net CS_PERIPH_3_5V: U11.11 (4Y)
- new net CS_RAM_0_3V: U12.2 (1A)
- new net CS_RAM_0_5V: U12.3 (1Y)
- new net CS_RAM_1_3V: U12.5 (2A)
- new net CS_RAM_1_5V: U12.6 (2Y)
- new net CS_RAM_2_3V: U12.9 (3A)
- new net CS_RAM_2_5V: U12.8 (3Y)
- new net CS_RAM_3_3V: U12.12 (4A)
- new net CS_RAM_3_5V: U12.11 (4Y)
