File: schematics/kicad/LVL_SHIFT_5_TO_3.sch (KiCad schematic (older format))
At the start: 4 parts

Commit message: Change a lot of things, especially pinning between sheets
Parts:
- added R5, R6: 10k, symbol R
- C29, C30: renamed from C?; value 0.1uF -> 1uF
- gave numbers to parts that had none: 2
Connections:
- net GND: now also R5.1, R6.1; no longer U13.19 (nOE), U14.19 (nOE)
- net INPUT_4_3V: now reaches U14.11 (B7)
- net INPUT_3_3V: now reaches U14.12 (B6)
- net INPUT_2_3V: now reaches U14.13 (B5)
- net INPUT_1_3V: now reaches U14.14 (B4)
- net INPUT_0_3V: now reaches U14.15 (B3)
- net INPUT_0_5V: now reaches U14.5 (A3)
- net INPUT_1_5V: now reaches U14.6 (A4)
- net INPUT_2_5V: now reaches U14.7 (A5)
- net INPUT_3_5V: now reaches U14.8 (A6)
- net INPUT_4_5V: now reaches U14.9 (A7)
- new net: R5.2, U13.19 (nOE)
- new net: R6.2, U14.19 (nOE)
Changed lines of the file:
@@
 LIBS:tinkerforge
 LIBS:shardy
+LIBS:XC1654CT-ND
+LIBS:XC1654CT
+LIBS:ld1117
+LIBS:ncp1117
+LIBS:CS8900A-CQ3Z
 LIBS:68k computer-cache
 EELAYER 25 0
@@
 $Descr A4 11693 8268
 encoding utf-8
-Sheet 8 9
+Sheet 5 7
 Title ""
 Date ""
@@
 $EndDescr
 $Comp
-L 74LVC245 U?
+L 74LVC245 U13
 U 1 1 5737E7C5
 P 2500 2150
-F 0 "U?" H 2350 2700 60  0000 C CNN
+F 0 "U13" H 2350 2700 60  0000 C CNN
 F 1 "74LVC245" H 2500 1600 60  0000 C CNN
 F 2 "" H 2500 2150 60  0000 C CNN
@@
 $EndComp
 $Comp
-L +3V3 #PWR?
+L +3V3 #PWR76
 U 1 1 5737E7FD
 P 2500 1350
-F 0 "#PWR?" H 2500 1200 50  0001 C CNN
+F 0 "#PWR76" H 2500 1200 50  0001 C CNN
 F 1 "+3V3" H 2500 1490 50  0000 C CNN
 F 2 "" H 2500 1350 50  0000 C CNN
@@
 $EndComp
 Wire Wire Line
-	1400 1350 2000 1350
-Wire Wire Line
-	2000 1350 2500 1350
-Wire Wire Line
-	2500 1350 3050 1350
+	1400 1350 3050 1350
 Wire Wire Line
 	2000 1350 2000 1700
@@
 	2000 2600 2000 2750
 $Comp
-L GND #PWR?
+L GND #PWR74
 U 1 1 5737E82B
 P 2000 2750
-F 0 "#PWR?" H 2000 2500 50  0001 C CNN
+F 0 "#PWR74" H 2000 2500 50  0001 C CNN
 F 1 "GND" H 2000 2600 50  0000 C CNN
 F 2 "" H 2000 2750 50  0000 C CNN
@@
 $EndComp
 Wire Wire Line
-	2850 1800 3500 1800
-Wire Wire Line
 	3500 1800 3500 1900
 $Comp
-L C C?
+L C C29
 U 1 1 5737E861
 P 1400 1550
-F 0 "C?" H 1425 1650 50  0000 L CNN
-F 1 "0.1uF" H 1425 1450 50  0000 L CNN
+F 0 "C29" H 1425 1650 50  0000 L CNN
+F 1 "1uF" H 1425 1450 50  0000 L CNN
 F 2 "" H 1438 1400 50  0000 C CNN
 F 3 "" H 1400 1550 50  0000 C CNN
@@
 	1400 1700 1400 1800
 $Comp
-L GND #PWR?
+L GND #PWR72
 U 1 1 5737E8CA
 P 1400 1800
-F 0 "#PWR?" H 1400 1550 50  0001 C CNN
+F 0 "#PWR72" H 1400 1550 50  0001 C CNN
 F 1 "GND" H 1400 1650 50  0000 C CNN
 F 2 "" H 1400 1800 50  0000 C CNN
@@
 	2850 2600 2950 2600
 $Comp
-L GND #PWR?
+L GND #PWR78
 U 1 1 5737EDDE
 P 3500 1900
-F 0 "#PWR?" H 3500 1650 50  0001 C CNN
+F 0 "#PWR78" H 3500 1650 50  0001 C CNN
 F 1 "GND" H 3500 1750 50  0000 C CNN
 F 2 "" H 3500 1900 50  0000 C CNN
@@
 $EndComp
 $Comp
-L 74LVC245 U?
+L 74LVC245 U14
 U 1 1 5737EE3D
 P 2500 3950
-F 0 "U?" H 2350 4500 60  0000 C CNN
+F 0 "U14" H 2350 4500 60  0000 C CNN
 F 1 "74LVC245" H 2500 3400 60  0000 C CNN
 F 2 "" H 2500 3950 60  0000 C CNN
@@
 $EndComp
 $Comp
-L +3V3 #PWR?
+L +3V3 #PWR77
 U 1 1 5737EE43
 P 2500 3150
-F 0 "#PWR?" H 2500 3000 50  0001 C CNN
+F 0 "#PWR77" H 2500 3000 50  0001 C CNN
 F 1 "+3V3" H 2500 3290 50  0000 C CNN
 F 2 "" H 2500 3150 50  0000 C CNN
@@
 $EndComp
 Wire Wire Line
-	1400 3150 2000 3150
-Wire Wire Line
-	2000 3150 2500 3150
-Wire Wire Line
-	2500 3150 3050 3150
+	1400 3150 3050 3150
 Wire Wire Line
 	2000 3150 2000 3500
@@
 	2000 4400 2000 4550
 $Comp
-L GND #PWR?
+L GND #PWR75
 U 1 1 5737EE51
 P 2000 4550
-F 0 "#PWR?" H 2000 4300 50  0001 C CNN
+F 0 "#PWR75" H 2000 4300 50  0001 C CNN
 F 1 "GND" H 2000 4400 50  0000 C CNN
 F 2 "" H 2000 4550 50  0000 C CNN
@@
 $EndComp
 Wire Wire Line
-	2850 3600 3500 3600
-Wire Wire Line
 	3500 3600 3500 3700
 $Comp
-L C C?
+L C C30
 U 1 1 5737EE59
 P 1400 3350
-F 0 "C?" H 1425 3450 50  0000 L CNN
-F 1 "0.1uF" H 1425 3250 50  0000 L CNN
+F 0 "C30" H 1425 3450 50  0000 L CNN
+F 1 "1uF" H 1425 3250 50  0000 L CNN
 F 2 "" H 1438 3200 50  0000 C CNN
 F 3 "" H 1400 3350 50  0000 C CNN
@@
 	1400 3500 1400 3600
 $Comp
-L GND #PWR?
+L GND #PWR73
 U 1 1 5737EE62
 P 1400 3600
-F 0 "#PWR?" H 1400 3350 50  0001 C CNN
+F 0 "#PWR73" H 1400 3350 50  0001 C CNN
 F 1 "GND" H 1400 3450 50  0000 C CNN
 F 2 "" H 1400 3600 50  0000 C CNN
@@
 Wire Wire Line
 	2150 3800 2050 3800
-Text HLabel 2950 3700 2    60   Output ~ 0
-FC0_3V
-Text HLabel 2950 3800 2    60   Output ~ 0
-FC1_3V
-Text HLabel 2950 3900 2    60   Output ~ 0
-FC2_3V
-Wire Wire Line
-	2850 3700 2950 3700
-Wire Wire Line
-	2850 3800 2950 3800
-Wire Wire Line
-	2850 3900 2950 3900
-$Comp
-L GND #PWR?
+$Comp
+L GND #PWR79
 U 1 1 5737EE88
 P 3500 3700
-F 0 "#PWR?" H 3500 3450 50  0001 C CNN
+F 0 "#PWR79" H 3500 3450 50  0001 C CNN
 F 1 "GND" H 3500 3550 50  0000 C CNN
 F 2 "" H 3500 3700 50  0000 C CNN
@@
 	1    0    0    -1
 $EndComp
+Wire Wire Line
+	2150 3900 2050 3900
+Wire Wire Line
+	2150 4000 2050 4000
+Wire Wire Line
+	2150 4100 2050 4100
+Wire Wire Line
+	2150 4200 2050 4200
+Wire Wire Line
+	2150 4300 2050 4300
+Text HLabel 2050 3900 0    60   Input ~ 0
+INPUT_0_5V
+Text HLabel 2050 4000 0    60   Input ~ 0
+INPUT_1_5V
+Text HLabel 2050 4100 0    60   Input ~ 0
+INPUT_2_5V
+Text HLabel 2050 4200 0    60   Input ~ 0
+INPUT_3_5V
+Text HLabel 2050 4300 0    60   Input ~ 0
+INPUT_4_5V
+Wire Wire Line
+	2850 3900 2950 3900
+Wire Wire Line
+	2850 3800 2950 3800
+Wire Wire Line
+	2850 3700 2950 3700
+Text HLabel 2950 3900 2    60   Output ~ 0
+FC2_3V
+Text HLabel 2950 3800 2    60   Output ~ 0
+FC1_3V
+Text HLabel 2950 3700 2    60   Output ~ 0
+FC0_3V
+Wire Wire Line
+	2850 4200 2950 4200
+Wire Wire Line
+	2850 4100 2950 4100
+Wire Wire Line
+	2850 4000 2950 4000
+Text HLabel 2950 4200 2    60   Output ~ 0
+INPUT_2_3V
+Text HLabel 2950 4100 2    60   Output ~ 0
+INPUT_1_3V
+Text HLabel 2950 4000 2    60   Output ~ 0
+INPUT_0_3V
+Wire Wire Line
+	2850 4400 2950 4400
+Wire Wire Line
+	2850 4300 2950 4300
+Text HLabel 2950 4400 2    60   Output ~ 0
+INPUT_4_3V
+Text HLabel 2950 4300 2    60   Output ~ 0
+INPUT_3_3V
+$Comp
+L R R6
+U 1 1 5757FA7B
+P 3150 3600
+F 0 "R6" V 3230 3600 50  0000 C CNN
+F 1 "10k" V 3150 3600 50  0000 C CNN
+F 2 "" V 3080 3600 50  0000 C CNN
+F 3 "" H 3150 3600 50  0000 C CNN
+	1    3150 3600
+	0    1    1    0
+$EndComp
+Wire Wire Line
+	2850 3600 3000 3600
+Wire Wire Line
+	3300 3600 3500 3600
+$Comp
+L R R5
+U 1 1 5757FB4D
+P 3100 1800
+F 0 "R5" V 3180 1800 50  0000 C CNN
+F 1 "10k" V 3100 1800 50  0000 C CNN
+F 2 "" V 3030 1800 50  0000 C CNN
+F 3 "" H 3100 1800 50  0000 C CNN
+	1    3100 1800
+	0    1    1    0
+$EndComp
+Wire Wire Line
+	2850 1800 2950 1800
+Wire Wire Line
+	3250 1800 3500 1800
 $EndSCHEMATC
